File: Board/Control Board.sch (EAGLE design)
At the start: 103 parts

Commit message: Made changes for v0.1.1
Removed two MOSFET boards and two voltage step-up/step-down boards. Reassigned MOSFET control pins.
Attempted to fix the 12V DC power barrel jack.
Added jumper header block for controlling enable pins on motor driver boards.
Tweaked positions of various components.
Added 12V power supply switch and LED indicator.
Added corner M3 mounting holes.
Improved silkscreen and added missing labels.
Parts:
- removed MOSFETIN7, MOSFETIN8, VCCREG7, VCCREG8: (no value), SparkFun-Connectors:CONN_05LOCK
- removed MOSFETVCC7, MOSFETVCC8: (no value), SparkFun-Connectors:CONN_03LOCK
- removed VCCEXT7, VCCEXT8: (no value), SparkFun-Connectors:CONN_022.54MM_SCREWTERM
- removed VCCOUT1: (no value), SparkFun-Connectors:CONN_04LOCK
- removed VCCOUT5: (no value), SparkFun-Connectors:CONN_04POLAR
- added 12VSWITCH: 4-1825136-5, 4-1825136-5:4-1825136-5
- added LED1: (no value), SparkFun-LED:LED3MM
- added LEDR1: (no value), SparkFun-Resistors:RESISTORAXIAL-0.3
- added STEPPERCTL1, STEPPEREN1, STEPPERGND1: (no value), SparkFun-Connectors:CONN_04LOCK
Connections:
- removed net EXTVCC7: MOSFETVCC7.1, VCCEXT7.2
- removed net EXTVCC8: MOSFETVCC8.1, VCCEXT8.2
- removed net MOSFETVCC7: MOSFETIN7.1, MOSFETIN7.2, MOSFETVCC7.2
- removed net MOSFETVCC8: MOSFETIN8.1, MOSFETIN8.2, MOSFETVCC8.2
- removed net REGVCC7: MOSFETVCC7.3, VCCOUT1.4, VCCOUT5.4, VCCREG7.1
- removed net REGVCC8: MOSFETVCC8.3, VCCOUT1.1, VCCOUT5.1, VCCREG8.1
- new net 12VSUPPLY: 12VIN.1, 12VOUT1.1, 12VOUT1.4, 12VOUT2.1, 12VOUT2.4, 12VSWITCH.1
- new net N$1: LED1.C, LEDR1.1
- new net STEPEN1: STEPPEREN1.1, STEPPERIN1.8
- new net STEPEN2: STEPPEREN1.2, STEPPERIN2.8
- new net STEPEN3: STEPPEREN1.3, STEPPERIN3.8
- new net STEPEN4: STEPPEREN1.4, STEPPERIN4.8
- net 12V: now also 12VSWITCH.2, LED1.A; no longer 12VIN.1, 12VOUT1.1, 12VOUT1.4, 12VOUT2.1, 12VOUT2.4, VCCREG7.3, VCCREG8.3
- net 38: now also STEPPERCTL1.1; no longer MOSFETIN8.5
- net 39: now also STEPPERCTL1.2; no longer MOSFETIN7.5
- net 40: now also STEPPERCTL1.3; no longer MOSFETIN6.5
- net 41: now also STEPPERCTL1.4; no longer MOSFETIN5.5
- net 42: no longer MOSFETIN4.5
- net 43: no longer MOSFETIN3.5
- net 44: no longer MOSFETIN2.5
- net 45: no longer MOSFETIN1.5
- net 48: now also MOSFETIN6.5
- net 49: now also MOSFETIN5.5
- net 50: now also MOSFETIN4.5
- net 51: now also MOSFETIN3.5
- net 52: now also MOSFETIN2.5
- net 53: now also MOSFETIN1.5
- net GND: now also 12VIN.2, LEDR1.2, STEPPERGND1.1, STEPPERGND1.2, STEPPERGND1.3, STEPPERGND1.4; no longer 12VIN.3, MOSFETIN7.3, MOSFETIN7.4, MOSFETIN8.3, MOSFETIN8.4, VCCEXT7.1, VCCEXT8.1, VCCOUT1.2, VCCOUT1.3, VCCOUT5.2, VCCOUT5.3, VCCREG7.2, VCCREG8.2
- net STEPUART1: now also STEPPERIN1.4
- net STEPUART2: now also STEPPERIN2.4
- net STEPUART3: now also STEPPERIN3.4
- net STEPUART4: now also STEPPERIN4.4
