File: ODSv1.0.0-BT/Backplane.sch (KiCad schematic (older format))
At the start: 38 parts

Commit message: Associate backplane template symbols with footprints and BOM info
Parts:
- D1, D2: footprint (none) -> LED_SMD:LED_0603_1608Metric; MPN (none) -> LTST-C190KSKT; Manufacturer (none) -> Lite-On; Ordering URL (none) -> https://www.digikey.com/en/products/detail/lite-on-inc/LTST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
- D3: footprint (none) -> LED_SMD:LED_0603_1608Metric; MPN (none) -> LTST-C190KFKT; Manufacturer (none) -> Lite-On; Ordering URL (none) -> https://www.digikey.com/en/products/detail/lite-on-inc/LTST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
- D4, D5: footprint (none) -> LED_SMD:LED_0603_1608Metric; MPN (none) -> LTST-C190KRKT; Manufacturer (none) -> Lite-On; Ordering URL (none) -> https://www.digikey.com/en/products/detail/lite-on-inc/LTST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
- D6, D7, D8: footprint (none) -> LED_SMD:LED_0603_1608Metric; MPN (none) -> LTST-C190TBKT; Manufacturer (none) -> Lite-On; Ordering URL (none) -> https://www.digikey.com/en/products/detail/lite-on-inc/LTST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
- R1, R3, R5: footprint (none) -> Resistor_SMD:R_1206_3216Metric_Pad1.42x1.75mm_HandSolder; MPN (none) -> RC1206FR-070RL; Manufacturer (none) -> Yageo; Ordering URL (none) -> https://www.digikey.com/en/products/detail/yageo/RC1206FR-0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
- R10, R11, R12, R13, R14, R15, R16, R17, R18, R19, R2, R20, R21, R22, R4, R6, R7, R8, R9: footprint (none) -> Resistor_SMD:R_1206_3216Metric_Pad1.42x1.75mm_HandSolder
- R23: footprint (none) -> Resistor_SMD:R_0603_1608Metric; MPN (none) -> RC0603FR-07270RL; Manufacturer (none) -> Yageo; Ordering URL (none) -> https://www.digikey.com/en/products/detail/yageo/RC0603FR-0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
- R24: footprint (none) -> Resistor_SMD:R_0603_1608Metric; MPN (none) -> RC0603FR-071KL; Manufacturer (none) -> Yageo; Ordering URL (none) -> https://www.digikey.com/en/products/detail/yageo/RC0603FR-0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
- R25: footprint (none) -> Resistor_SMD:R_0603_1608Metric; MPN (none) -> RC0603FR-071K2L; Manufacturer (none) -> Yageo; Ordering URL (none) -> https://www.digikey.com/en/products/detail/yageo/RC0603FR-0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
- R26, R27: footprint (none) -> Resistor_SMD:R_0603_1608Metric; MPN (none) -> RC0603FR-07560RL; Manufacturer (none) -> Yageo; Ordering URL (none) -> https://www.digikey.com/en/products/detail/yageo/RC0603FR-0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
- R28: footprint (none) -> Resistor_SMD:R_0603_1608Metric; MPN (none) -> RC0603FR-07150RL; Manufacturer (none) -> Yageo; Ordering URL (none) -> https://www.digikey.com/en/products/detail/yageo/RC0603FR-0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
- R29, R30: footprint (none) -> Resistor_SMD:R_0603_1608Metric; MPN (none) -> RC0603FR-0775RL; Manufacturer (none) -> Yageo; Ordering URL (none) -> https://www.digikey.com/en/products/detail/yageo/RC0603FR-0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

Commit message: Remap pins for easier layout
Parts:
- removed R1, R3, R5: 0, Resistor_SMD:R_1206_3216Metric_Pad1.42x1.75mm_HandSolder, symbol Device:R
- removed R2, R22, R4, R6: DNP, Resistor_SMD:R_1206_3216Metric_Pad1.42x1.75mm_HandSolder, symbol Device:R
- renumbered D6 to D1, D7 to D2, D8 to D3, D1 to D4, D2 to D5, D3 to D6, D4 to D7, D5 to D8, R7 to R1, R16 to R10, R17 to R11, R18 to R12, R19 to R13, R20 to R14, R21 to R15, R23 to R16, R24 to R17, R25 to R18, R26 to R19, R8 to R2, R27 to R20, R28 to R21, R29 to R22, R30 to R23, R9 to R3, R10 to R4, R11 to R5, R12 to R6, R13 to R7, R14 to R8, R15 to R9
Connections:
- wire segments 179 -> 160
Other:
- note added: "Customization Instructions:\n- Select a DSCS pin to use for selecting SPI devices on the plane, by changing a resistor from DNP\n to 0 for the corresponding DSCS pin in the "SPI DSCS Selector" section.\n- If you don't need one of the power supplies, change the corresponding LED value and resistor value\n in the "Power Indicator LEDs" section to DNP.\n- Customize the colors and order of programmab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"
- note added: "Use the other SPI bus in\nthe default BOM by\nchanging the nets."
- note removed: "Customization Instructions:\nSelect a DSCS pin to use for selecting SPI devices on the plane, by changing a resistor\nfrom DNP to 0 for the corresponding DSCS pin in the "SPI DSCS Selector" section.\nCustomize the colors and order of programmable indicator LEDs in the\n"Programmable Indicator LEDs" section; make sure to update resistor values.\nIf you need to use any pins from the GPIO or Interpl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"
- note removed: "Use the other SPI bus in\nthe default BOM by flipping\nthe resistor values."
- moved on the sheet: D1, D2, D3, R16, R17, R18
