File: ODSv1.0.0-BT/Backplane.sch (KiCad schematic (older format))
At the start: 31 parts

Commit message: Prepare BOM properties for assembly
Parts:
- D1, D2, D3, D4, D5, D6, D7, D8: Assembly Notes (none) -> Polarity is indicated by a diode symbol either next to the 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; Type (none) -> SMD
- R16, R17, R18, R19, R20, R21, R22, R23: Type (none) -> SMD
Changed lines of the file:
@@
 F 5 "Yageo" H 9000 4550 50  0001 C CNN "Manufacturer"
 F 6 "https://www.digikey.com/en/products/detail/yageo/RC0603FR-07560RL/727304" H 9000 4550 50  0001 C CNN "Ordering URL"
+F 7 "SMD" H 9000 4550 50  0001 C CNN "Type"
 	1    9000 4550
 	0    1    1    0
@@
 F 5 "Yageo" H 9000 4650 50  0001 C CNN "Manufacturer"
 F 6 "https://www.digikey.com/en/products/detail/yageo/RC0603FR-07560RL/727304" H 9000 4650 50  0001 C CNN "Ordering URL"
+F 7 "SMD" H 9000 4650 50  0001 C CNN "Type"
 	1    9000 4650
 	0    1    1    0
@@
 F 5 "Yageo" H 9000 4750 50  0001 C CNN "Manufacturer"
 F 6 "https://www.digikey.com/en/products/detail/yageo/RC0603FR-07150RL/726958" H 9000 4750 50  0001 C CNN "Ordering URL"
+F 7 "SMD" H 9000 4750 50  0001 C CNN "Type"
 	1    9000 4750
 	0    1    1    0
@@
 F 5 "Yageo" H 9000 4850 50  0001 C CNN "Manufacturer"
 F 6 "https://www.digikey.com/en/products/detail/yageo/RC0603FR-0775RL/727377" H 9000 4850 50  0001 C CNN "Ordering URL"
+F 7 "SMD" H 9000 4850 50  0001 C CNN "Type"
 	1    9000 4850
 	0    1    1    0
@@
 F 5 "Yageo" H 9000 4950 50  0001 C CNN "Manufacturer"
 F 6 "https://www.digikey.com/en/products/detail/yageo/RC0603FR-0775RL/727377" H 9000 4950 50  0001 C CNN "Ordering URL"
+F 7 "SMD" H 9000 4950 50  0001 C CNN "Type"
 	1    9000 4950
 	0    1    1    0
@@
 F 5 "Lite-On" H 8550 4950 50  0001 C CNN "Manufacturer"
 F 6 "https://www.digikey.com/en/products/detail/lite-on-inc/LTST-C190KRKT/386817" H 8550 4950 50  0001 C CNN "Ordering URL"
+F 7 "SMD" H 8550 4950 50  0001 C CNN "Type"
+F 8 "Polarity is indicated by a diode symbol either next to the LED or at the end of the line of LEDs." H 8550 4950 50  0001 C CNN "Assembly Notes"
 	1    8550 4950
 	1    0    0    1
@@
 F 5 "Lite-On" H 8550 4850 50  0001 C CNN "Manufacturer"
 F 6 "https://www.digikey.com/en/products/detail/lite-on-inc/LTST-C190KRKT/386817" H 8550 4850 50  0001 C CNN "Ordering URL"
+F 7 "SMD" H 8550 4850 50  0001 C CNN "Type"
+F 8 "Polarity is indicated by a diode symbol either next to the LED or at the end of the line of LEDs." H 8550 4850 50  0001 C CNN "Assembly Notes"
 	1    8550 4850
 	1    0    0    1
@@
 F 5 "Lite-On" H 8550 4750 50  0001 C CNN "Manufacturer"
 F 6 "https://www.digikey.com/en/products/detail/lite-on-inc/LTST-C190KFKT/386813" H 8550 4750 50  0001 C CNN "Ordering URL"
+F 7 "SMD" H 8550 4750 50  0001 C CNN "Type"
+F 8 "Polarity is indicated by a diode symbol either next to the LED or at the end of the line of LEDs." H 8550 4750 50  0001 C CNN "Assembly Notes"
 	1    8550 4750
 	1    0    0    1
@@
 F 5 "Lite-On" H 8550 4650 50  0001 C CNN "Manufacturer"
 F 6 "https://www.digikey.com/en/products/detail/lite-on-inc/LTST-C190KSKT/386819" H 8550 4650 50  0001 C CNN "Ordering URL"
+F 7 "SMD" H 8550 4650 50  0001 C CNN "Type"
+F 8 "Polarity is indicated by a diode symbol either next to the LED or at the end of the line of LEDs." H 8550 4650 50  0001 C CNN "Assembly Notes"
 	1    8550 4650
 	1    0    0    1
@@
 F 5 "Lite-On" H 8550 4550 50  0001 C CNN "Manufacturer"
 F 6 "https://www.digikey.com/en/products/detail/lite-on-inc/LTST-C190KSKT/386819" H 8550 4550 50  0001 C CNN "Ordering URL"
+F 7 "SMD" H 8550 4550 50  0001 C CNN "Type"
+F 8 "Polarity is indicated by a diode symbol either next to the LED or at the end of the line of LEDs." H 8550 4550 50  0001 C CNN "Assembly Notes"
 	1    8550 4550
 	1    0    0    1
@@
 F 5 "Lite-On" H 4450 6100 50  0001 C CNN "Manufacturer"
 F 6 "https://www.digikey.com/en/products/detail/lite-on-inc/LTST-C190TBKT/388529" H 4450 6100 50  0001 C CNN "Ordering URL"
+F 7 "SMD" H 4450 6100 50  0001 C CNN "Type"
+F 8 "Polarity is indicated by a diode symbol either next to the LED or at the end of the line of LEDs." H 4450 6100 50  0001 C CNN "Assembly Notes"
 	1    4450 6100
 	1    0    0    1
@@
 F 5 "Yageo" H 4850 6100 50  0001 C CNN "Manufacturer"
 F 6 "https://www.digikey.com/en/products/detail/yageo/RC0603FR-07270RL/727103" H 4850 6100 50  0001 C CNN "Ordering URL"
+F 7 "SMD" H 4850 6100 50  0001 C CNN "Type"
 	1    4850 6100
 	0    -1   1    0
@@
 F 5 "Lite-On" H 4450 6200 50  0001 C CNN "Manufacturer"
 F 6 "https://www.digikey.com/en/products/detail/lite-on-inc/LTST-C190TBKT/388529" H 4450 6200 50  0001 C CNN "Ordering URL"
+F 7 "SMD" H 4450 6200 50  0001 C CNN "Type"
+F 8 "Polarity is indicated by a diode symbol either next to the LED or at the end of the line of LEDs." H 4450 6200 50  0001 C CNN "Assembly Notes"
 	1    4450 6200
 	1    0    0    1
@@
 F 5 "Yageo" H 4850 6200 50  0001 C CNN "Manufacturer"
 F 6 "https://www.digikey.com/en/products/detail/yageo/RC0603FR-071KL/726843" H 4850 6200 50  0001 C CNN "Ordering URL"
+F 7 "SMD" H 4850 6200 50  0001 C CNN "Type"
 	1    4850 6200
 	0    -1   1    0
@@
 F 5 "Lite-On" H 4450 6300 50  0001 C CNN "Manufacturer"
 F 6 "https://www.digikey.com/en/products/detail/lite-on-inc/LTST-C190TBKT/388529" H 4450 6300 50  0001 C CNN "Ordering URL"
+F 7 "SMD" H 4450 6300 50  0001 C CNN "Type"
+F 8 "Polarity is indicated by a diode symbol either next to the LED or at the end of the line of LEDs." H 4450 6300 50  0001 C CNN "Assembly Notes"
 	1    4450 6300
 	1    0    0    1
@@
 F 5 "Yageo" H 4850 6300 50  0001 C CNN "Manufacturer"
 F 6 "https://www.digikey.com/en/products/detail/yageo/RC0603FR-071K2L/726852" H 4850 6300 50  0001 C CNN "Ordering URL"
+F 7 "SMD" H 4850 6300 50  0001 C CNN "Type"
 	1    4850 6300
 	0    -1   1    0

Commit message: Add Digikey part number as BOM field for Digkey's BOM manager
Parts:
- D1, D2, D3: Digikey ID (none) -> 160-1646-1-ND
- D4, D5: Digikey ID (none) -> 160-1437-1-ND
- D6: Digikey ID (none) -> 160-1434-1-ND
- D7, D8: Digikey ID (none) -> 160-1436-1-ND
- R16: Digikey ID (none) -> 311-270HRCT-ND
- R17: Digikey ID (none) -> 311-1.00KHRCT-ND
- R18: Digikey ID (none) -> 311-1.20KHRCT-ND
- R19, R20: Digikey ID (none) -> 311-560HRCT-ND
- R21: Digikey ID (none) -> 311-150HRCT-ND
- R22, R23: Digikey ID (none) -> 311-75.0HRCT-ND
Changed lines of the file:
@@
 F 6 "https://www.digikey.com/en/products/detail/yageo/RC0603FR-07560RL/727304" H 9000 4550 50  0001 C CNN "Ordering URL"
 F 7 "SMD" H 9000 4550 50  0001 C CNN "Type"
+F 8 "311-560HRCT-ND" H 9000 4550 50  0001 C CNN "Digikey ID"
 	1    9000 4550
 	0    1    1    0
@@
 F 6 "https://www.digikey.com/en/products/detail/yageo/RC0603FR-07560RL/727304" H 9000 4650 50  0001 C CNN "Ordering URL"
 F 7 "SMD" H 9000 4650 50  0001 C CNN "Type"
+F 8 "311-560HRCT-ND" H 9000 4650 50  0001 C CNN "Digikey ID"
 	1    9000 4650
 	0    1    1    0
@@
 F 6 "https://www.digikey.com/en/products/detail/yageo/RC0603FR-07150RL/726958" H 9000 4750 50  0001 C CNN "Ordering URL"
 F 7 "SMD" H 9000 4750 50  0001 C CNN "Type"
+F 8 "311-150HRCT-ND" H 9000 4750 50  0001 C CNN "Digikey ID"
 	1    9000 4750
 	0    1    1    0
@@
 F 6 "https://www.digikey.com/en/products/detail/yageo/RC0603FR-0775RL/727377" H 9000 4850 50  0001 C CNN "Ordering URL"
 F 7 "SMD" H 9000 4850 50  0001 C CNN "Type"
+F 8 "311-75.0HRCT-ND" H 9000 4850 50  0001 C CNN "Digikey ID"
 	1    9000 4850
 	0    1    1    0
@@
 F 6 "https://www.digikey.com/en/products/detail/yageo/RC0603FR-0775RL/727377" H 9000 4950 50  0001 C CNN "Ordering URL"
 F 7 "SMD" H 9000 4950 50  0001 C CNN "Type"
+F 8 "311-75.0HRCT-ND" H 9000 4950 50  0001 C CNN "Digikey ID"
 	1    9000 4950
 	0    1    1    0
@@
 F 7 "SMD" H 8550 4950 50  0001 C CNN "Type"
 F 8 "Polarity is indicated by a diode symbol either next to the LED or at the end of the line of LEDs." H 8550 4950 50  0001 C CNN "Assembly Notes"
+F 9 "160-1436-1-ND" H 8550 4950 50  0001 C CNN "Digikey ID"
 	1    8550 4950
 	1    0    0    1
@@
 F 7 "SMD" H 8550 4850 50  0001 C CNN "Type"
 F 8 "Polarity is indicated by a diode symbol either next to the LED or at the end of the line of LEDs." H 8550 4850 50  0001 C CNN "Assembly Notes"
+F 9 "160-1436-1-ND" H 8550 4850 50  0001 C CNN "Digikey ID"
 	1    8550 4850
 	1    0    0    1
@@
 F 7 "SMD" H 8550 4750 50  0001 C CNN "Type"
 F 8 "Polarity is indicated by a diode symbol either next to the LED or at the end of the line of LEDs." H 8550 4750 50  0001 C CNN "Assembly Notes"
+F 9 "160-1434-1-ND" H 8550 4750 50  0001 C CNN "Digikey ID"
 	1    8550 4750
 	1    0    0    1
@@
 F 7 "SMD" H 8550 4650 50  0001 C CNN "Type"
 F 8 "Polarity is indicated by a diode symbol either next to the LED or at the end of the line of LEDs." H 8550 4650 50  0001 C CNN "Assembly Notes"
+F 9 "160-1437-1-ND" H 8550 4650 50  0001 C CNN "Digikey ID"
 	1    8550 4650
 	1    0    0    1
@@
 F 7 "SMD" H 8550 4550 50  0001 C CNN "Type"
 F 8 "Polarity is indicated by a diode symbol either next to the LED or at the end of the line of LEDs." H 8550 4550 50  0001 C CNN "Assembly Notes"
+F 9 "160-1437-1-ND" H 8550 4550 50  0001 C CNN "Digikey ID"
 	1    8550 4550
 	1    0    0    1
@@
 F 7 "SMD" H 4450 6100 50  0001 C CNN "Type"
 F 8 "Polarity is indicated by a diode symbol either next to the LED or at the end of the line of LEDs." H 4450 6100 50  0001 C CNN "Assembly Notes"
+F 9 "160-1646-1-ND" H 4450 6100 50  0001 C CNN "Digikey ID"
 	1    4450 6100
 	1    0    0    1
@@
 F 6 "https://www.digikey.com/en/products/detail/yageo/RC0603FR-07270RL/727103" H 4850 6100 50  0001 C CNN "Ordering URL"
 F 7 "SMD" H 4850 6100 50  0001 C CNN "Type"
+F 8 "311-270HRCT-ND" H 4850 6100 50  0001 C CNN "Digikey ID"
 	1    4850 6100
 	0    -1   1    0
@@
 F 7 "SMD" H 4450 6200 50  0001 C CNN "Type"
 F 8 "Polarity is indicated by a diode symbol either next to the LED or at the end of the line of LEDs." H 4450 6200 50  0001 C CNN "Assembly Notes"
+F 9 "160-1646-1-ND" H 4450 6200 50  0001 C CNN "Digikey ID"
 	1    4450 6200
 	1    0    0    1
@@
 F 6 "https://www.digikey.com/en/products/detail/yageo/RC0603FR-071KL/726843" H 4850 6200 50  0001 C CNN "Ordering URL"
 F 7 "SMD" H 4850 6200 50  0001 C CNN "Type"
+F 8 "311-1.00KHRCT-ND" H 4850 6200 50  0001 C CNN "Digikey ID"
 	1    4850 6200
 	0    -1   1    0
@@
 F 7 "SMD" H 4450 6300 50  0001 C CNN "Type"
 F 8 "Polarity is indicated by a diode symbol either next to the LED or at the end of the line of LEDs." H 4450 6300 50  0001 C CNN "Assembly Notes"
+F 9 "160-1646-1-ND" H 4450 6300 50  0001 C CNN "Digikey ID"
 	1    4450 6300
 	1    0    0    1
@@
 F 6 "https://www.digikey.com/en/products/detail/yageo/RC0603FR-071K2L/726852" H 4850 6300 50  0001 C CNN "Ordering URL"
 F 7 "SMD" H 4850 6300 50  0001 C CNN "Type"
+F 8 "311-1.20KHRCT-ND" H 4850 6300 50  0001 C CNN "Digikey ID"
 	1    4850 6300
 	0    -1   1    0
