File: ODSv1.0.0-BT/Connectors.sch (KiCad schematic (older format))
At the start: 2 parts, among them J1 Conn_02x60_Odd_Even, J2 Conn_02x60_Odd_Even

Commit message: Prepare BOM properties for assembly
Parts:
- J1, J2: Assembly Notes (none) -> Pin 1 is indicated by a triangle on the component and an ex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; Type (none) -> SMD
Changed lines of the file:
@@
 F 5 "Hirose" H 2450 3950 50  0001 C CNN "Manufacturer"
 F 6 "https://www.digikey.com/en/products/detail/hirose-electric-co-ltd/FX20-120P-0-5SV15/3461671" H 2450 3950 50  0001 C CNN "Ordering URL"
+F 7 "SMD" H 2450 3950 50  0001 C CNN "Type"
+F 8 "Pin 1 is indicated by a triangle on the component and an extra line in the silkscreen." H 2450 3950 50  0001 C CNN "Assembly Notes"
 	1    2450 3950
 	1    0    0    -1
@@
 F 5 "Hirose" H 5450 3950 50  0001 C CNN "Manufacturer"
 F 6 "https://www.digikey.com/en/products/detail/hirose-electric-co-ltd/FX20-120S-0-5SV/3461673" H 5450 3950 50  0001 C CNN "Ordering URL"
+F 7 "SMD" H 5450 3950 50  0001 C CNN "Type"
+F 8 "Pin 1 is indicated by a triangle on the component and an extra line in the silkscreen." H 5450 3950 50  0001 C CNN "Assembly Notes"
 	1    5450 3950
 	1    0    0    -1

Commit message: Add Digikey part number as BOM field for Digkey's BOM manager
Parts:
- J1: Digikey ID (none) -> H12043-ND
- J2: Digikey ID (none) -> H12041-ND
Changed lines of the file:
@@
 F 7 "SMD" H 2450 3950 50  0001 C CNN "Type"
 F 8 "Pin 1 is indicated by a triangle on the component and an extra line in the silkscreen." H 2450 3950 50  0001 C CNN "Assembly Notes"
+F 9 "H12043-ND" H 2450 3950 50  0001 C CNN "Digikey ID"
 	1    2450 3950
 	1    0    0    -1
@@
 F 7 "SMD" H 5450 3950 50  0001 C CNN "Type"
 F 8 "Pin 1 is indicated by a triangle on the component and an extra line in the silkscreen." H 5450 3950 50  0001 C CNN "Assembly Notes"
+F 9 "H12041-ND" H 5450 3950 50  0001 C CNN "Digikey ID"
 	1    5450 3950
 	1    0    0    -1

Commit message: Add LICENSE files and README text, and rename backplane to backbone
Parts:
- J1: footprint Backplane_Connector_Hirose:Hirose_FX20_FX20-120P-0.5SV_2x60_P0.50mm_Vertical -> Backbone_Connector_Hirose:Hirose_FX20_FX20-120P-0.5SV_2x60_P0.50mm_Vertical; symbol Backplane_Connector_Generic:Conn_02x60_Odd_Even -> Backbone_Connector_Generic:Conn_02x60_Odd_Even
- J2: footprint Backplane_Connector_Hirose:Hirose_FX20_FX20-120S-0.5SV_2x60_P0.50mm_Vertical -> Backbone_Connector_Hirose:Hirose_FX20_FX20-120S-0.5SV_2x60_P0.50mm_Vertical; symbol Backplane_Connector_Generic:Conn_02x60_Odd_Even -> Backbone_Connector_Generic:Conn_02x60_Odd_Even
Changed lines of the file:
@@
 encoding utf-8
 Sheet 4 4
-Title "Backplane Template"
-Date "2020-12-26"
+Title "Backbone Template"
+Date "2021-01-19"
 Rev "v0.1.0"
 Comp "Prakash Lab/Octopi Team"
@@
 $EndDescr
 $Comp
-L Backplane_Connector_Generic:Conn_02x60_Odd_Even J?
+L Backbone_Connector_Generic:Conn_02x60_Odd_Even J?
 U 1 1 60EAE366
 P 2450 3950
@@
 F 0 "J1" H 2500 7067 50  0000 C CNN
 F 1 "Conn_02x60_Odd_Even" H 2500 6976 50  0000 C CNN
-F 2 "Backplane_Connector_Hirose:Hirose_FX20_FX20-120P-0.5SV_2x60_P0.50mm_Vertical" H 2450 3950 50  0001 C CNN
+F 2 "Backbone_Connector_Hirose:Hirose_FX20_FX20-120P-0.5SV_2x60_P0.50mm_Vertical" H 2450 3950 50  0001 C CNN
 F 3 "https://www.hirose.com/product/document?clcode=&productname=&series=FX20&documenttype=Catalog&lang=en&documentid=D49373_en" H 2450 3950 50  0001 C CNN
 F 4 "FX20-120P-0.5SV15" H 2450 3950 50  0001 C CNN "MPN"
@@
 $EndComp
 $Comp
-L Backplane_Connector_Generic:Conn_02x60_Odd_Even J?
+L Backbone_Connector_Generic:Conn_02x60_Odd_Even J?
 U 1 1 61296724
 P 5450 3950
@@
 F 0 "J2" H 5500 7067 50  0000 C CNN
 F 1 "Conn_02x60_Odd_Even" H 5500 6976 50  0000 C CNN
-F 2 "Backplane_Connector_Hirose:Hirose_FX20_FX20-120S-0.5SV_2x60_P0.50mm_Vertical" H 5450 3950 50  0001 C CNN
+F 2 "Backbone_Connector_Hirose:Hirose_FX20_FX20-120S-0.5SV_2x60_P0.50mm_Vertical" H 5450 3950 50  0001 C CNN
 F 3 "https://www.hirose.com/product/document?clcode=&productname=&series=FX20&documenttype=Catalog&lang=en&documentid=D49373_en" H 5450 3950 50  0001 C CNN
 F 4 "FX20-120S-0.5SV" H 5450 3950 50  0001 C CNN "MPN"
