File: ODSv1.0.0-BT/ODSv1.0.0-BT.sch (KiCad schematic (older format))
At the start: 4 parts

Commit message: Fix implementation of SPI CS multiplexing system (#22)
* Disconnect PP-T41's MAX7317's DOUT, since it's not needed anyways (#16)

* Disconnect BT & BP-Jmp backbone MAX7317 DOUT (#16); make DOUT output pin

* Replace DAC with a second MAX7317 expander with pullup resistors

* Insert 3-state buffers between MAX7317 DOUTs and CIPO in BP-Jmp (#16)

* Update symbol fields for I/O expansion components in BP-Jmp

* Consolidate free space by moving the AD7689 chip

* Add pull-ups on demuxed DCS (#17), move pull-ups to bottom of BP-Jmp

* Insert 3-state buffers between all MAX7317 DOUTs and CIPO (#16)

* Add bypass caps to the 3-state buffers for BP-Jmp's I/O expanders

* Fix title block for SPI DCS Selector sheet in BP-Jmp

* Use 2k pullups instead of 20k pullups on BP-Jmp

* Add 2k pullups on demuxed DSCS pins in PP-T41

* Define a NoPufferfish BOM variant of PP-T41

* Adjust the 12V copper fills on PP-T41

* Add 2k pullups within the DSCS selector in PP-T41 (#17)

* Add more information to READMEs

* Add 2k pullups within DCS selectors (#17), bump BP-Jmp to 0.2.0

* Fix errors in PR template for modified boards

* Move usage on I/O peripherals into a subsection in BP-Jmp's README.md

* Update KiCad preview & mechanical renders of all boards

* Improve & consolidate pull request templates

* Update raytrace renders of the entire stack

* Add missing definition for NoPufferfish variant for PP-T41

* Add link to CADLab project for this repo

* Remove the message annoyingly added by CADLab to top of README.md
Changed lines of the file:
@@
 Sheet 1 4
 Title "Backbone Template"
-Date "2021-03-09"
+Date "2021-03-11"
 Rev "v0.1.1"
 Comp "Prakash Lab/Octopi Team"
@@
 F0 "Backbone" 50
 F1 "Backbone.sch" 50
-F2 "SPI_SCK" O R 1750 1450 50
-F3 "SPI_COPI" O R 1750 1550 50
-F4 "SPI_CIPO" T R 1750 1650 50
+F2 "SPI0_SCK" O R 1750 1450 50
+F3 "SPI0_COPI" O R 1750 1550 50
+F4 "SPI0_CIPO" T R 1750 1650 50
 F5 "3.3V" O R 1750 1050 50
 F6 "5V" O R 1750 1150 50
