File: ODSv1.0.0-PP-T41/Backplane.sch (KiCad schematic (older format))
At the start: 16 parts

Commit message: Prepare BOM properties for assembly
Parts:
- D1, D2, D3, D4, D5, D6, D7, D8: Assembly Notes (none) -> Polarity is indicated by a diode symbol either next to the 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; Type (none) -> SMD
- R10, R11, R12, R13, R14, R7, R8, R9: Type (none) -> SMD
Changed lines of the file:
@@
 F 5 "Yageo" H 7500 4700 50  0001 C CNN "Manufacturer"
 F 6 "https://www.digikey.com/en/products/detail/yageo/RC0603FR-07560RL/727304" H 7500 4700 50  0001 C CNN "Ordering URL"
+F 7 "SMD" H 7500 4700 50  0001 C CNN "Type"
 	1    7500 4700
 	0    1    1    0
@@
 F 5 "Yageo" H 7500 4800 50  0001 C CNN "Manufacturer"
 F 6 "https://www.digikey.com/en/products/detail/yageo/RC0603FR-07560RL/727304" H 7500 4800 50  0001 C CNN "Ordering URL"
+F 7 "SMD" H 7500 4800 50  0001 C CNN "Type"
 	1    7500 4800
 	0    1    1    0
@@
 F 5 "Yageo" H 7500 4900 50  0001 C CNN "Manufacturer"
 F 6 "https://www.digikey.com/en/products/detail/yageo/RC0603FR-07150RL/726958" H 7500 4900 50  0001 C CNN "Ordering URL"
+F 7 "SMD" H 7500 4900 50  0001 C CNN "Type"
 	1    7500 4900
 	0    1    1    0
@@
 F 5 "Yageo" H 7500 5000 50  0001 C CNN "Manufacturer"
 F 6 "https://www.digikey.com/en/products/detail/yageo/RC0603FR-0775RL/727377" H 7500 5000 50  0001 C CNN "Ordering URL"
+F 7 "SMD" H 7500 5000 50  0001 C CNN "Type"
 	1    7500 5000
 	0    1    1    0
@@
 F 5 "Yageo" H 7500 5100 50  0001 C CNN "Manufacturer"
 F 6 "https://www.digikey.com/en/products/detail/yageo/RC0603FR-0775RL/727377" H 7500 5100 50  0001 C CNN "Ordering URL"
+F 7 "SMD" H 7500 5100 50  0001 C CNN "Type"
 	1    7500 5100
 	0    1    1    0
@@
 F 5 "Lite-On" H 7050 5100 50  0001 C CNN "Manufacturer"
 F 6 "https://www.digikey.com/en/products/detail/lite-on-inc/LTST-C190KRKT/386817" H 7050 5100 50  0001 C CNN "Ordering URL"
+F 7 "SMD" H 7050 5100 50  0001 C CNN "Type"
+F 8 "Polarity is indicated by a diode symbol either next to the LED or at the end of the line of LEDs." H 7050 5100 50  0001 C CNN "Assembly Notes"
 	1    7050 5100
 	1    0    0    1
@@
 F 5 "Lite-On" H 7050 5000 50  0001 C CNN "Manufacturer"
 F 6 "https://www.digikey.com/en/products/detail/lite-on-inc/LTST-C190KRKT/386817" H 7050 5000 50  0001 C CNN "Ordering URL"
+F 7 "SMD" H 7050 5000 50  0001 C CNN "Type"
+F 8 "Polarity is indicated by a diode symbol either next to the LED or at the end of the line of LEDs." H 7050 5000 50  0001 C CNN "Assembly Notes"
 	1    7050 5000
 	1    0    0    1
@@
 F 5 "Lite-On" H 7050 4900 50  0001 C CNN "Manufacturer"
 F 6 "https://www.digikey.com/en/products/detail/lite-on-inc/LTST-C190KFKT/386813" H 7050 4900 50  0001 C CNN "Ordering URL"
+F 7 "SMD" H 7050 4900 50  0001 C CNN "Type"
+F 8 "Polarity is indicated by a diode symbol either next to the LED or at the end of the line of LEDs." H 7050 4900 50  0001 C CNN "Assembly Notes"
 	1    7050 4900
 	1    0    0    1
@@
 F 5 "Lite-On" H 7050 4800 50  0001 C CNN "Manufacturer"
 F 6 "https://www.digikey.com/en/products/detail/lite-on-inc/LTST-C190KSKT/386819" H 7050 4800 50  0001 C CNN "Ordering URL"
+F 7 "SMD" H 7050 4800 50  0001 C CNN "Type"
+F 8 "Polarity is indicated by a diode symbol either next to the LED or at the end of the line of LEDs." H 7050 4800 50  0001 C CNN "Assembly Notes"
 	1    7050 4800
 	1    0    0    1
@@
 F 5 "Lite-On" H 7050 4700 50  0001 C CNN "Manufacturer"
 F 6 "https://www.digikey.com/en/products/detail/lite-on-inc/LTST-C190KSKT/386819" H 7050 4700 50  0001 C CNN "Ordering URL"
+F 7 "SMD" H 7050 4700 50  0001 C CNN "Type"
+F 8 "Polarity is indicated by a diode symbol either next to the LED or at the end of the line of LEDs." H 7050 4700 50  0001 C CNN "Assembly Notes"
 	1    7050 4700
 	1    0    0    1
@@
 F 5 "Lite-On" H 2200 6150 50  0001 C CNN "Manufacturer"
 F 6 "https://www.digikey.com/en/products/detail/lite-on-inc/LTST-C190TBKT/388529" H 2200 6150 50  0001 C CNN "Ordering URL"
+F 7 "SMD" H 2200 6150 50  0001 C CNN "Type"
+F 8 "Polarity is indicated by a diode symbol either next to the LED or at the end of the line of LEDs." H 2200 6150 50  0001 C CNN "Assembly Notes"
 	1    2200 6150
 	1    0    0    1
@@
 F 5 "Yageo" H 2600 6150 50  0001 C CNN "Manufacturer"
 F 6 "https://www.digikey.com/en/products/detail/yageo/RC0603FR-07270RL/727103" H 2600 6150 50  0001 C CNN "Ordering URL"
+F 7 "SMD" H 2600 6150 50  0001 C CNN "Type"
 	1    2600 6150
 	0    -1   1    0
@@
 F 5 "Lite-On" H 2200 6250 50  0001 C CNN "Manufacturer"
 F 6 "https://www.digikey.com/en/products/detail/lite-on-inc/LTST-C190TBKT/388529" H 2200 6250 50  0001 C CNN "Ordering URL"
+F 7 "SMD" H 2200 6250 50  0001 C CNN "Type"
+F 8 "Polarity is indicated by a diode symbol either next to the LED or at the end of the line of LEDs." H 2200 6250 50  0001 C CNN "Assembly Notes"
 	1    2200 6250
 	1    0    0    1
@@
 F 5 "Yageo" H 2600 6250 50  0001 C CNN "Manufacturer"
 F 6 "https://www.digikey.com/en/products/detail/yageo/RC0603FR-071KL/726843" H 2600 6250 50  0001 C CNN "Ordering URL"
+F 7 "SMD" H 2600 6250 50  0001 C CNN "Type"
 	1    2600 6250
 	0    -1   1    0
@@
 F 5 "Lite-On" H 2200 6350 50  0001 C CNN "Manufacturer"
 F 6 "https://www.digikey.com/en/products/detail/lite-on-inc/LTST-C190TBKT/388529" H 2200 6350 50  0001 C CNN "Ordering URL"
+F 7 "SMD" H 2200 6350 50  0001 C CNN "Type"
+F 8 "Polarity is indicated by a diode symbol either next to the LED or at the end of the line of LEDs." H 2200 6350 50  0001 C CNN "Assembly Notes"
 	1    2200 6350
 	1    0    0    1
@@
 F 5 "Yageo" H 2600 6350 50  0001 C CNN "Manufacturer"
 F 6 "https://www.digikey.com/en/products/detail/yageo/RC0603FR-071K2L/726852" H 2600 6350 50  0001 C CNN "Ordering URL"
+F 7 "SMD" H 2600 6350 50  0001 C CNN "Type"
 	1    2600 6350
 	0    -1   1    0

Commit message: Add Digikey part number as BOM field for Digkey's BOM manager
Parts:
- D1, D2, D3: Digikey ID (none) -> 160-1646-1-ND
- D4, D5: Digikey ID (none) -> 160-1437-1-ND
- D6: Digikey ID (none) -> 160-1434-1-ND
- D7, D8: Digikey ID (none) -> 160-1436-1-ND
- R10, R11: Digikey ID (none) -> 311-560HRCT-ND
- R12: Digikey ID (none) -> 311-150HRCT-ND
- R13, R14: Digikey ID (none) -> 311-75.0HRCT-ND
- R7: Digikey ID (none) -> 311-270HRCT-ND
- R8: Digikey ID (none) -> 311-1.00KHRCT-ND
Changed lines of the file:
@@
 F 6 "https://www.digikey.com/en/products/detail/yageo/RC0603FR-07560RL/727304" H 7500 4700 50  0001 C CNN "Ordering URL"
 F 7 "SMD" H 7500 4700 50  0001 C CNN "Type"
+F 8 "311-560HRCT-ND" H 7500 4700 50  0001 C CNN "Digikey ID"
 	1    7500 4700
 	0    1    1    0
@@
 F 6 "https://www.digikey.com/en/products/detail/yageo/RC0603FR-07560RL/727304" H 7500 4800 50  0001 C CNN "Ordering URL"
 F 7 "SMD" H 7500 4800 50  0001 C CNN "Type"
+F 8 "311-560HRCT-ND" H 7500 4800 50  0001 C CNN "Digikey ID"
 	1    7500 4800
 	0    1    1    0
@@
 F 6 "https://www.digikey.com/en/products/detail/yageo/RC0603FR-07150RL/726958" H 7500 4900 50  0001 C CNN "Ordering URL"
 F 7 "SMD" H 7500 4900 50  0001 C CNN "Type"
+F 8 "311-150HRCT-ND" H 7500 4900 50  0001 C CNN "Digikey ID"
 	1    7500 4900
 	0    1    1    0
@@
 F 6 "https://www.digikey.com/en/products/detail/yageo/RC0603FR-0775RL/727377" H 7500 5000 50  0001 C CNN "Ordering URL"
 F 7 "SMD" H 7500 5000 50  0001 C CNN "Type"
+F 8 "311-75.0HRCT-ND" H 7500 5000 50  0001 C CNN "Digikey ID"
 	1    7500 5000
 	0    1    1    0
@@
 F 6 "https://www.digikey.com/en/products/detail/yageo/RC0603FR-0775RL/727377" H 7500 5100 50  0001 C CNN "Ordering URL"
 F 7 "SMD" H 7500 5100 50  0001 C CNN "Type"
+F 8 "311-75.0HRCT-ND" H 7500 5100 50  0001 C CNN "Digikey ID"
 	1    7500 5100
 	0    1    1    0
@@
 F 7 "SMD" H 7050 5100 50  0001 C CNN "Type"
 F 8 "Polarity is indicated by a diode symbol either next to the LED or at the end of the line of LEDs." H 7050 5100 50  0001 C CNN "Assembly Notes"
+F 9 "160-1436-1-ND" H 7050 5100 50  0001 C CNN "Digikey ID"
 	1    7050 5100
 	1    0    0    1
@@
 F 7 "SMD" H 7050 5000 50  0001 C CNN "Type"
 F 8 "Polarity is indicated by a diode symbol either next to the LED or at the end of the line of LEDs." H 7050 5000 50  0001 C CNN "Assembly Notes"
+F 9 "160-1436-1-ND" H 7050 5000 50  0001 C CNN "Digikey ID"
 	1    7050 5000
 	1    0    0    1
@@
 F 7 "SMD" H 7050 4900 50  0001 C CNN "Type"
 F 8 "Polarity is indicated by a diode symbol either next to the LED or at the end of the line of LEDs." H 7050 4900 50  0001 C CNN "Assembly Notes"
+F 9 "160-1434-1-ND" H 7050 4900 50  0001 C CNN "Digikey ID"
 	1    7050 4900
 	1    0    0    1
@@
 F 7 "SMD" H 7050 4800 50  0001 C CNN "Type"
 F 8 "Polarity is indicated by a diode symbol either next to the LED or at the end of the line of LEDs." H 7050 4800 50  0001 C CNN "Assembly Notes"
+F 9 "160-1437-1-ND" H 7050 4800 50  0001 C CNN "Digikey ID"
 	1    7050 4800
 	1    0    0    1
@@
 F 7 "SMD" H 7050 4700 50  0001 C CNN "Type"
 F 8 "Polarity is indicated by a diode symbol either next to the LED or at the end of the line of LEDs." H 7050 4700 50  0001 C CNN "Assembly Notes"
+F 9 "160-1437-1-ND" H 7050 4700 50  0001 C CNN "Digikey ID"
 	1    7050 4700
 	1    0    0    1
@@
 F 7 "SMD" H 2200 6150 50  0001 C CNN "Type"
 F 8 "Polarity is indicated by a diode symbol either next to the LED or at the end of the line of LEDs." H 2200 6150 50  0001 C CNN "Assembly Notes"
+F 9 "160-1646-1-ND" H 2200 6150 50  0001 C CNN "Digikey ID"
 	1    2200 6150
 	1    0    0    1
@@
 F 6 "https://www.digikey.com/en/products/detail/yageo/RC0603FR-07270RL/727103" H 2600 6150 50  0001 C CNN "Ordering URL"
 F 7 "SMD" H 2600 6150 50  0001 C CNN "Type"
+F 8 "311-270HRCT-ND" H 2600 6150 50  0001 C CNN "Digikey ID"
 	1    2600 6150
 	0    -1   1    0
@@
 F 7 "SMD" H 2200 6250 50  0001 C CNN "Type"
 F 8 "Polarity is indicated by a diode symbol either next to the LED or at the end of the line of LEDs." H 2200 6250 50  0001 C CNN "Assembly Notes"
+F 9 "160-1646-1-ND" H 2200 6250 50  0001 C CNN "Digikey ID"
 	1    2200 6250
 	1    0    0    1
@@
 F 6 "https://www.digikey.com/en/products/detail/yageo/RC0603FR-071KL/726843" H 2600 6250 50  0001 C CNN "Ordering URL"
 F 7 "SMD" H 2600 6250 50  0001 C CNN "Type"
+F 8 "311-1.00KHRCT-ND" H 2600 6250 50  0001 C CNN "Digikey ID"
 	1    2600 6250
 	0    -1   1    0
@@
 F 7 "SMD" H 2200 6350 50  0001 C CNN "Type"
 F 8 "Polarity is indicated by a diode symbol either next to the LED or at the end of the line of LEDs." H 2200 6350 50  0001 C CNN "Assembly Notes"
+F 9 "160-1646-1-ND" H 2200 6350 50  0001 C CNN "Digikey ID"
 	1    2200 6350
 	1    0    0    1
