File: ODSv1.0.0-PP-T41/SPIDSCSSelector.sch (KiCad schematic (older format))
At the start: 4 parts, among them U1 MAX7317, U2 74HC4067PW

Commit message: Prepare BOM properties for assembly
Parts:
- C1, C2, U1, U2: Type (none) -> SMD
Changed lines of the file:
@@
 F 5 "Maxim" H 2000 2100 50  0001 C CNN "Manufacturer"
 F 6 "https://www.digikey.com/en/products/detail/maxim-integrated/MAX7317AEE-T/1781026" H 2000 2100 50  0001 C CNN "Ordering URL"
+F 7 "SMD" H 2000 2100 50  0001 C CNN "Type"
 	1    2000 2100
 	1    0    0    -1
@@
 F 5 "Nexperia" H 4750 1900 50  0001 C CNN "Manufacturer"
 F 6 "https://www.digikey.com/en/products/detail/nexperia-usa-inc/74HC4067PW118/1230424" H 4750 1900 50  0001 C CNN "Ordering URL"
+F 7 "SMD" H 4750 1900 50  0001 C CNN "Type"
 	1    4750 1900
 	1    0    0    -1
@@
 F 5 "AVX" H 2750 1150 50  0001 C CNN "Manufacturer"
 F 6 "https://www.digikey.com/en/products/detail/avx-corporation/06033C473KAT2A/563345" H 2750 1150 50  0001 C CNN "Ordering URL"
+F 7 "SMD" H 2750 1150 50  0001 C CNN "Type"
 	1    2750 1150
 	1    0    0    -1
@@
 F 5 "AVX" H 3500 1150 50  0001 C CNN "Manufacturer"
 F 6 "https://www.digikey.com/en/products/detail/avx-corporation/06033C104KAT4A/3247517" H 3500 1150 50  0001 C CNN "Ordering URL"
+F 7 "SMD" H 3500 1150 50  0001 C CNN "Type"
 	1    3500 1150
 	1    0    0    -1

Commit message: Add Digikey part number as BOM field for Digkey's BOM manager
Parts:
- C1: Digikey ID (none) -> 478-1235-1-ND
- C2: Digikey ID (none) -> 478-7018-1-ND
- U1: Digikey ID (none) -> MAX7317AEE+TCT-ND
- U2: Digikey ID (none) -> 1727-2042-1-ND
Changed lines of the file:
@@
 F 6 "https://www.digikey.com/en/products/detail/maxim-integrated/MAX7317AEE-T/1781026" H 2000 2100 50  0001 C CNN "Ordering URL"
 F 7 "SMD" H 2000 2100 50  0001 C CNN "Type"
+F 8 "MAX7317AEE+TCT-ND" H 2000 2100 50  0001 C CNN "Digikey ID"
 	1    2000 2100
 	1    0    0    -1
@@
 F 6 "https://www.digikey.com/en/products/detail/nexperia-usa-inc/74HC4067PW118/1230424" H 4750 1900 50  0001 C CNN "Ordering URL"
 F 7 "SMD" H 4750 1900 50  0001 C CNN "Type"
+F 8 "1727-2042-1-ND" H 4750 1900 50  0001 C CNN "Digikey ID"
 	1    4750 1900
 	1    0    0    -1
@@
 F 6 "https://www.digikey.com/en/products/detail/avx-corporation/06033C473KAT2A/563345" H 2750 1150 50  0001 C CNN "Ordering URL"
 F 7 "SMD" H 2750 1150 50  0001 C CNN "Type"
+F 8 "478-1235-1-ND" H 2750 1150 50  0001 C CNN "Digikey ID"
 	1    2750 1150
 	1    0    0    -1
@@
 F 6 "https://www.digikey.com/en/products/detail/avx-corporation/06033C104KAT4A/3247517" H 3500 1150 50  0001 C CNN "Ordering URL"
 F 7 "SMD" H 3500 1150 50  0001 C CNN "Type"
+F 8 "478-7018-1-ND" H 3500 1150 50  0001 C CNN "Digikey ID"
 	1    3500 1150
 	1    0    0    -1
