File: ODSv1.0.0-PP-T41/Teensy.sch (KiCad schematic (older format))
At the start: 2 parts, among them J3 Conn_01x24, J4 Conn_01x24

Commit message: Prepare BOM properties for assembly
Parts:
- J3, J4: Type (none) -> SMD
Changed lines of the file:
@@
 F 6 "Samtec" H 2450 2100 50  0001 C CNN "Manufacturer"
 F 7 "https://www.digikey.com/en/products/detail/samtec-inc/SSW-124-22-F-S-VS/7893884" H 2450 2100 50  0001 C CNN "Ordering URL"
+F 8 "SMD" H 2450 2100 50  0001 C CNN "Type"
 	1    2450 2100
 	1    0    0    -1
@@
 F 6 "Samtec" H 4050 2200 50  0001 C CNN "Manufacturer"
 F 7 "https://www.digikey.com/en/products/detail/samtec-inc/SSW-124-22-F-S-VS/7893884" H 4050 2200 50  0001 C CNN "Ordering URL"
+F 8 "SMD" H 4050 2200 50  0001 C CNN "Type"
 	1    4050 2200
 	-1   0    0    1

Commit message: Add Digikey part number as BOM field for Digkey's BOM manager
Parts:
- J3, J4: Digikey ID (none) -> SSW-124-22-F-S-VS-ND
Changed lines of the file:
@@
 F 7 "https://www.digikey.com/en/products/detail/samtec-inc/SSW-124-22-F-S-VS/7893884" H 2450 2100 50  0001 C CNN "Ordering URL"
 F 8 "SMD" H 2450 2100 50  0001 C CNN "Type"
+F 9 "SSW-124-22-F-S-VS-ND" H 2450 2100 50  0001 C CNN "Digikey ID"
 	1    2450 2100
 	1    0    0    -1
@@
 F 7 "https://www.digikey.com/en/products/detail/samtec-inc/SSW-124-22-F-S-VS/7893884" H 4050 2200 50  0001 C CNN "Ordering URL"
 F 8 "SMD" H 4050 2200 50  0001 C CNN "Type"
+F 9 "SSW-124-22-F-S-VS-ND" H 4050 2200 50  0001 C CNN "Digikey ID"
 	1    4050 2200
 	-1   0    0    1
