File: ODSv1.0.0-PP-T41/Teensy.sch (KiCad schematic (older format))
At the start: 2 parts, among them J3 Conn_01x24, J4 Conn_01x24

Commit message: Make minor improvements to PP-T41 (#20)
* Fix 3D models for Teensy 4.1 and female headers to mount it (#18)

* Add header as test points for signal not exposed on the backbone (#15)
Parts:
- J3, J4: footprint Connector_PinHeader_2.54mm:PinHeader_1x24_P2.54mm_Vertical_SMD_Pin1Left -> Connector_PinSocket_2.54mm:PinSocket_1x24_P2.54mm_Vertical_SMD_Pin1Left
Changed lines of the file:
@@
 $Descr USLetter 11000 8500
 encoding utf-8
-Sheet 5 7
+Sheet 5 8
 Title "Processing Plane for Teensy 4.1"
-Date "2021-02-07"
+Date "2021-03-09"
 Rev "v0.1.1"
 Comp "Prakash Lab/Octopi Team"
@@
 F 0 "J3" H 2530 2092 50  0000 L CNN
 F 1 "Conn_01x24" H 2530 2001 50  0000 L CNN
-F 2 "Connector_PinHeader_2.54mm:PinHeader_1x24_P2.54mm_Vertical_SMD_Pin1Left" H 2450 2100 50  0001 C CNN
+F 2 "Connector_PinSocket_2.54mm:PinSocket_1x24_P2.54mm_Vertical_SMD_Pin1Left" H 2450 2100 50  0001 C CNN
 F 3 "http://suddendocs.samtec.com/catalog_english/ssw_sm.pdf" H 2450 2100 50  0001 C CNN
 F 4 "Teensy 4.1" H 2450 2100 50  0001 C CNN "Associated Board"
@@
 F 0 "J4" H 3968 775 50  0000 C CNN
 F 1 "Conn_01x24" H 3968 866 50  0000 C CNN
-F 2 "Connector_PinHeader_2.54mm:PinHeader_1x24_P2.54mm_Vertical_SMD_Pin1Left" H 4050 2200 50  0001 C CNN
+F 2 "Connector_PinSocket_2.54mm:PinSocket_1x24_P2.54mm_Vertical_SMD_Pin1Left" H 4050 2200 50  0001 C CNN
 F 3 "http://suddendocs.samtec.com/catalog_english/ssw_sm.pdf" H 4050 2200 50  0001 C CNN
 F 4 "Teensy 4.1" H 4050 2200 50  0001 C CNN "Associated Board"
