File: ODSv1.0.0-BP-Jmp/SPIDCSSelector.sch (KiCad schematic (older format))
At the start: 4 parts, among them U1 MAX7317, U2 74HC4067PW

Commit message: Update READMEs, and update customization instructions in BT
Parts:
- U2: Config (none) -> -NoExpansion
Changed lines of the file:
@@
 F 7 "SMD" H 4750 1900 50  0001 C CNN "Type"
 F 8 "1727-2042-1-ND" H 4750 1900 50  0001 C CNN "Digikey ID"
+F 9 "-NoExpansion" H 4750 1900 50  0001 C CNN "Config"
 	1    4750 1900
 	1    0    0    -1
