File: ODSv1.0.0-BP-Jmp/SPIDCSSelector.sch (KiCad schematic (older format))
At the start: 4 parts, among them U1 MAX7317, U2 74HC4067PW

Commit message: Define a no-IC variant of BP-Jmp
Parts:
- U1: Config (none) -> -NoIC
- U2: Config -NoExpansion -> -NoExpansion, -NoIC
Changed lines of the file:
@@
 F 7 "SMD" H 2000 2100 50  0001 C CNN "Type"
 F 8 "MAX7317AEE+TCT-ND" H 2000 2100 50  0001 C CNN "Digikey ID"
+F 9 "-NoIC" H 2000 2100 50  0001 C CNN "Config"
 	1    2000 2100
 	1    0    0    -1
@@
 F 7 "SMD" H 4750 1900 50  0001 C CNN "Type"
 F 8 "1727-2042-1-ND" H 4750 1900 50  0001 C CNN "Digikey ID"
-F 9 "-NoExpansion" H 4750 1900 50  0001 C CNN "Config"
+F 9 "-NoExpansion, -NoIC" H 4750 1900 50  0001 C CNN "Config"
 	1    4750 1900
 	1    0    0    -1

Commit message: Fix problems with BP-Jmp variant configurations
Parts:
- C1, C2: Config (none) -> -NoIC
- U2: Config -NoExpansion, -NoIC -> -NoIC
Changed lines of the file:
@@
 F 7 "SMD" H 4750 1900 50  0001 C CNN "Type"
 F 8 "1727-2042-1-ND" H 4750 1900 50  0001 C CNN "Digikey ID"
-F 9 "-NoExpansion, -NoIC" H 4750 1900 50  0001 C CNN "Config"
+F 9 "-NoIC" H 4750 1900 50  0001 C CNN "Config"
 	1    4750 1900
 	1    0    0    -1
@@
 F 7 "SMD" H 2750 1200 50  0001 C CNN "Type"
 F 8 "478-1235-1-ND" H 2750 1200 50  0001 C CNN "Digikey ID"
+F 9 "-NoIC" H 2750 1200 50  0001 C CNN "Config"
 	1    2750 1200
 	1    0    0    -1
@@
 F 7 "SMD" H 3500 1150 50  0001 C CNN "Type"
 F 8 "478-7018-1-ND" H 3500 1150 50  0001 C CNN "Digikey ID"
+F 9 "-NoIC" H 3500 1150 50  0001 C CNN "Config"
 	1    3500 1150
 	1    0    0    -1

Commit message: Fix implementation of SPI CS multiplexing system (#22)
* Disconnect PP-T41's MAX7317's DOUT, since it's not needed anyways (#16)

* Disconnect BT & BP-Jmp backbone MAX7317 DOUT (#16); make DOUT output pin

* Replace DAC with a second MAX7317 expander with pullup resistors

* Insert 3-state buffers between MAX7317 DOUTs and CIPO in BP-Jmp (#16)

* Update symbol fields for I/O expansion components in BP-Jmp

* Consolidate free space by moving the AD7689 chip

* Add pull-ups on demuxed DCS (#17), move pull-ups to bottom of BP-Jmp

* Insert 3-state buffers between all MAX7317 DOUTs and CIPO (#16)

* Add bypass caps to the 3-state buffers for BP-Jmp's I/O expanders

* Fix title block for SPI DCS Selector sheet in BP-Jmp

* Use 2k pullups instead of 20k pullups on BP-Jmp

* Add 2k pullups on demuxed DSCS pins in PP-T41

* Define a NoPufferfish BOM variant of PP-T41

* Adjust the 12V copper fills on PP-T41

* Add 2k pullups within the DSCS selector in PP-T41 (#17)

* Add more information to READMEs

* Add 2k pullups within DCS selectors (#17), bump BP-Jmp to 0.2.0

* Fix errors in PR template for modified boards

* Move usage on I/O peripherals into a subsection in BP-Jmp's README.md

* Update KiCad preview & mechanical renders of all boards

* Improve & consolidate pull request templates

* Update raytrace renders of the entire stack

* Add missing definition for NoPufferfish variant for PP-T41

* Add link to CADLab project for this repo

* Remove the message annoyingly added by CADLab to top of README.md
Parts:
- added C3: 0.1uF, Capacitor_SMD:C_0603_1608Metric, symbol Device:C
- added R16, R17, R18, R19, R20: 2k, Resistor_SMD:R_0603_1608Metric, symbol Device:R
- added U3: NC7SZ125, Package_TO_SOT_SMD:SOT-353_SC-70-5, symbol Octopi:NC7SZ125
Connections:
- net CIPO: now also U3.4; no longer U1.14 (DOUT)
- net GND: now also C3.2, U3.3 (GND)
- net ~DSCS~: now also U3.1
- net ~MUX_E~: now reaches U1.3 (P0), U2.15 (~E)
- net ~MUX_E~: now also R16.1
- net MUX_S0: now reaches U1.4 (P1), U2.10 (S0)
- net MUX_S0: now also R17.1
- net MUX_S1: now reaches U1.5 (P2), U2.11 (S1)
- net MUX_S1: now also R18.1
- net MUX_S2: now reaches U1.6 (P3), U2.14 (S2)
- net MUX_S2: now also R19.1
- net MUX_S3: now reaches U1.7 (P4), U2.13 (S3)
- net MUX_S3: now also R20.1
- net 3.3V renamed VCC
- net VCC: now also C3.1, R16.2, R17.2, R18.2, R19.2, R20.2, U3.5 (VCC)
- new net EXP_DOUT: U1.14 (DOUT), U3.2
Other:
- moved on the sheet: C1, C2, U1, U2
