File: ODSv1.0.0-BP-Jmp/IO Expander.sch (KiCad schematic (older format))
At the start: 10 parts, among them J20 Conn_02x10_Odd_Even, J21 Conn_02x10_Odd_Even, J22 Conn_02x10_Odd_Even, U3 MAX7317, U4 DACx0508xRTE

Commit message: Fix footprint and add 3D model for DAC80508, add docs for ICs
Parts:
- U4: footprint Package_DFN_QFN:Texas_S-PWQFN-N16_EP2.1x2.1mm_ThermalVias -> Package_DFN_QFN:WQFN-16-1EP_3x3mm_P0.5mm_EP1.6x1.6mm_ThermalVias
Changed lines of the file:
@@
 F 0 "U4" H 2200 4050 50  0000 L CNN
 F 1 "DACx0508xRTE" H 2150 3950 50  0000 R CNN
-F 2 "Package_DFN_QFN:Texas_S-PWQFN-N16_EP2.1x2.1mm_ThermalVias" H 2500 3000 50  0001 C CNN
+F 2 "Package_DFN_QFN:WQFN-16-1EP_3x3mm_P0.5mm_EP1.6x1.6mm_ThermalVias" H 2500 3000 50  0001 C CNN
 F 3 "https://www.ti.com/lit/ds/symlink/dac60508.pdf" H 2500 3550 50  0001 C CNN
 	1    2500 3500

Commit message: Add an ADC
Parts:
- added C10, C8, C9: 0.1uF, Capacitor_SMD:C_0603_1608Metric, symbol Device:C
- added C11: 10uF, Capacitor_SMD:C_0805_2012Metric, symbol Device:C
- added U5: AD7689xCP, Package_CSP:LFCSP-20-1EP_4x4mm_P0.5mm_EP2.5x2.5mm, symbol Analog_ADC:AD7689xCP
- C6: footprint Capacitor_SMD:C_0603_1608Metric -> Capacitor_SMD:C_0805_2012Metric; Digikey ID 478-10046-1-ND -> 478-10578-1-ND; MPN 06033C105KAT2A -> 0805ZC106KAT2A; Ordering URL https://www.digikey.com/en/products/detail/avx-corporation/06033C105KAT2A/6564240 -> https://www.digikey.com/en/products/detail/avx-corporation/0805ZC106KAT2A/3081418
Connections:
- net 3.3V: now also C8.1, C9.1, U5.1 (VDD), U5.15 (VIO), U5.20 (VDD)
- net GND: now also J22.19 (Pin_19), C10.2, C11.2, C8.2, C9.2, U5.21 (EPAD), U5.4 (GND), U5.5 (GND)
- net SPI0_CIPO: now also U5.14 (SDO)
- net SPI0_COPI: now also U5.12 (DIN)
- net SPI0_SCK: now also U5.13 (SCK)
- net ADCCOM: now reaches J22.1 (Pin_1)
- net ADCCOM: now also J22.11 (Pin_11), J22.13 (Pin_13), J22.15 (Pin_15), J22.17 (Pin_17), J22.3 (Pin_3), J22.5 (Pin_5), J22.7 (Pin_7), J22.9 (Pin_9), U5.10 (COM)
- net ADC4: now reaches J22.10 (Pin_10)
- net ADC4: now also U5.6 (IN4)
- net ADC5: now reaches J22.12 (Pin_12)
- net ADC5: now also U5.7 (IN5)
- net ADC6: now reaches J22.14 (Pin_14)
- net ADC6: now also U5.8 (IN6)
- net ADC7: now reaches J22.16 (Pin_16)
- net ADC7: now also U5.9 (IN7)
- net REF: now reaches J22.18 (Pin_18)
- net REF: now also C11.1, U5.2 (REF)
- net ADC0: now reaches J22.2 (Pin_2)
- net ADC0: now also U5.16 (IN0)
- net REFIN: now reaches J22.20 (Pin_20)
- net REFIN: now also C10.1, U5.3 (REFIN)
- net ADC1: now reaches J22.4 (Pin_4)
- net ADC1: now also U5.17 (IN1)
- net ADC2: now reaches J22.6 (Pin_6)
- net ADC2: now also U5.18 (IN2)
- net ADC3: now reaches J22.8 (Pin_8)
- net ADC3: now also U5.19 (IN3)
- new net ~DCS2~: U5.11 (CNV)
Other:
- moved on the sheet: C3, J22

Commit message: Update READMEs, and update customization instructions in BT
Parts:
- J20, J21, J22, U3, U4, U5: Config (none) -> -NoExpansion
Changed lines of the file:
@@
 F 7 "SMD" H 2500 1750 50  0001 C CNN "Type"
 F 8 "MAX7317AEE+TCT-ND" H 2500 1750 50  0001 C CNN "Digikey ID"
+F 9 "-NoExpansion" H 2500 1750 50  0001 C CNN "Config"
 	1    2500 1750
 	1    0    0    -1
@@
 F 2 "Connector_PinHeader_2.54mm:PinHeader_2x10_P2.54mm_Vertical_SMD" H 3950 1700 50  0001 C CNN
 F 3 "~" H 3950 1700 50  0001 C CNN
+F 4 "-NoExpansion" H 3950 1700 50  0001 C CNN "Config"
 	1    3950 1700
 	1    0    0    -1
@@
 F 2 "Package_DFN_QFN:WQFN-16-1EP_3x3mm_P0.5mm_EP1.6x1.6mm_ThermalVias" H 2500 3000 50  0001 C CNN
 F 3 "https://www.ti.com/lit/ds/symlink/dac60508.pdf" H 2500 3550 50  0001 C CNN
+F 4 "-NoExpansion" H 2500 3500 50  0001 C CNN "Config"
 	1    2500 3500
 	1    0    0    -1
@@
 F 2 "Connector_PinHeader_2.54mm:PinHeader_2x10_P2.54mm_Vertical_SMD" H 4050 3400 50  0001 C CNN
 F 3 "~" H 4050 3400 50  0001 C CNN
+F 4 "-NoExpansion" H 4050 3400 50  0001 C CNN "Config"
 	1    4050 3400
 	-1   0    0    -1
@@
 F 2 "Connector_PinHeader_2.54mm:PinHeader_2x10_P2.54mm_Vertical_SMD" H 9800 3400 50  0001 C CNN
 F 3 "~" H 9800 3400 50  0001 C CNN
+F 4 "-NoExpansion" H 9800 3400 50  0001 C CNN "Config"
 	1    9800 3400
 	-1   0    0    -1
@@
 F 2 "Package_CSP:LFCSP-20-1EP_4x4mm_P0.5mm_EP2.5x2.5mm" H 8500 3500 50  0001 C CNN
 F 3 "https://www.analog.com/media/en/technical-documentation/data-sheets/AD7682_7689.pdf" H 8500 3500 50  0001 C CNN
+F 4 "-NoExpansion" H 8500 3500 50  0001 C CNN "Config"
 	1    8500 3500
 	-1   0    0    -1

Commit message: Update BOM
Parts:
- J20, J21, J22: Digikey ID (none) -> SAM8990-ND; MPN (none) -> TSM-110-01-T-DV; Manufacturer (none) -> Samtec; Ordering URL (none) -> https://www.digikey.com/en/products/detail/samtec-inc/TSM-1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; Type (none) -> SMD
- U4: Digikey ID (none) -> 296-51047-1-ND; MPN (none) -> DAC80508ZRTER; Manufacturer (none) -> Texas Instruments; Ordering URL (none) -> https://www.digikey.com/en/products/detail/texas-instrument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; Type (none) -> SMD
- U5: Digikey ID (none) -> AD7689BCPZRL7CT-ND; MPN (none) -> AD7689BCPZRL7; Manufacturer (none) -> Analog Devices; Ordering URL (none) -> https://www.digikey.com/en/products/detail/analog-devices-i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; Type (none) -> SMD
Changed lines of the file:
@@
 F 1 "Conn_02x10_Odd_Even" H 4000 2250 50  0000 C CNN
 F 2 "Connector_PinHeader_2.54mm:PinHeader_2x10_P2.54mm_Vertical_SMD" H 3950 1700 50  0001 C CNN
-F 3 "~" H 3950 1700 50  0001 C CNN
+F 3 "http://suddendocs.samtec.com/catalog_english/tsm.pdf" H 3950 1700 50  0001 C CNN
 F 4 "-NoExpansion" H 3950 1700 50  0001 C CNN "Config"
+F 5 "SAM8990-ND" H 3950 1700 50  0001 C CNN "Digikey ID"
+F 6 "TSM-110-01-T-DV" H 3950 1700 50  0001 C CNN "MPN"
+F 7 "Samtec" H 3950 1700 50  0001 C CNN "Manufacturer"
+F 8 "https://www.digikey.com/en/products/detail/samtec-inc/TSM-110-01-T-DV/1236604" H 3950 1700 50  0001 C CNN "Ordering URL"
+F 9 "SMD" H 3950 1700 50  0001 C CNN "Type"
 	1    3950 1700
 	1    0    0    -1
@@
 F 3 "https://www.ti.com/lit/ds/symlink/dac60508.pdf" H 2500 3550 50  0001 C CNN
 F 4 "-NoExpansion" H 2500 3500 50  0001 C CNN "Config"
+F 5 "296-51047-1-ND" H 2500 3500 50  0001 C CNN "Digikey ID"
+F 6 "DAC80508ZRTER" H 2500 3500 50  0001 C CNN "MPN"
+F 7 "Texas Instruments" H 2500 3500 50  0001 C CNN "Manufacturer"
+F 8 "https://www.digikey.com/en/products/detail/texas-instruments/DAC80508ZRTER/9659605" H 2500 3500 50  0001 C CNN "Ordering URL"
+F 9 "SMD" H 2500 3500 50  0001 C CNN "Type"
 	1    2500 3500
 	1    0    0    -1
@@
 F 1 "Conn_02x10_Odd_Even" H 4100 3950 50  0000 C CNN
 F 2 "Connector_PinHeader_2.54mm:PinHeader_2x10_P2.54mm_Vertical_SMD" H 4050 3400 50  0001 C CNN
-F 3 "~" H 4050 3400 50  0001 C CNN
+F 3 "http://suddendocs.samtec.com/catalog_english/tsm.pdf" H 4050 3400 50  0001 C CNN
 F 4 "-NoExpansion" H 4050 3400 50  0001 C CNN "Config"
+F 5 "SAM8990-ND" H 4050 3400 50  0001 C CNN "Digikey ID"
+F 6 "TSM-110-01-T-DV" H 4050 3400 50  0001 C CNN "MPN"
+F 7 "Samtec" H 4050 3400 50  0001 C CNN "Manufacturer"
+F 8 "https://www.digikey.com/en/products/detail/samtec-inc/TSM-110-01-T-DV/1236604" H 4050 3400 50  0001 C CNN "Ordering URL"
+F 9 "SMD" H 4050 3400 50  0001 C CNN "Type"
 	1    4050 3400
 	-1   0    0    -1
@@
 F 1 "Conn_02x10_Odd_Even" H 9850 3950 50  0000 C CNN
 F 2 "Connector_PinHeader_2.54mm:PinHeader_2x10_P2.54mm_Vertical_SMD" H 9800 3400 50  0001 C CNN
-F 3 "~" H 9800 3400 50  0001 C CNN
+F 3 "http://suddendocs.samtec.com/catalog_english/tsm.pdf" H 9800 3400 50  0001 C CNN
 F 4 "-NoExpansion" H 9800 3400 50  0001 C CNN "Config"
+F 5 "SAM8990-ND" H 9800 3400 50  0001 C CNN "Digikey ID"
+F 6 "TSM-110-01-T-DV" H 9800 3400 50  0001 C CNN "MPN"
+F 7 "Samtec" H 9800 3400 50  0001 C CNN "Manufacturer"
+F 8 "https://www.digikey.com/en/products/detail/samtec-inc/TSM-110-01-T-DV/1236604" H 9800 3400 50  0001 C CNN "Ordering URL"
+F 9 "SMD" H 9800 3400 50  0001 C CNN "Type"
 	1    9800 3400
 	-1   0    0    -1
@@
 F 3 "https://www.analog.com/media/en/technical-documentation/data-sheets/AD7682_7689.pdf" H 8500 3500 50  0001 C CNN
 F 4 "-NoExpansion" H 8500 3500 50  0001 C CNN "Config"
+F 5 "AD7689BCPZRL7CT-ND" H 8500 3500 50  0001 C CNN "Digikey ID"
+F 6 "AD7689BCPZRL7" H 8500 3500 50  0001 C CNN "MPN"
+F 7 "Analog Devices" H 8500 3500 50  0001 C CNN "Manufacturer"
+F 8 "https://www.digikey.com/en/products/detail/analog-devices-inc/AD7689BCPZRL7/1873540" H 8500 3500 50  0001 C CNN "Ordering URL"
+F 9 "SMD" H 8500 3500 50  0001 C CNN "Type"
 	1    8500 3500
 	-1   0    0    -1
