File: ODSv1.0.0-BP-Jmp/Power Breakout.sch (KiCad schematic (older format))
At the start: 3 parts, among them J4 Conn_02x10_Odd_Even, J5 Conn_02x10_Odd_Even, J6 Conn_02x10_Odd_Even

Commit message: Update BOM
Parts:
- J4, J5, J6: Digikey ID (none) -> SAM15910-ND; MPN (none) -> TSM-110-01-T-DH; Manufacturer (none) -> Samtec; Ordering URL (none) -> https://www.digikey.com/en/products/detail/samtec-inc/TSM-1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; Type (none) -> SMD
Changed lines of the file:
@@
 F 1 "Conn_02x10_Odd_Even" H 2250 1950 50  0000 C CNN
 F 2 "Octopi:Samtec_TSM-110-01-X-DH_2x10_P2.54mm_Horizontal" H 2200 1400 50  0001 C CNN
-F 3 "~" H 2200 1400 50  0001 C CNN
+F 3 "http://suddendocs.samtec.com/catalog_english/tsm.pdf" H 2200 1400 50  0001 C CNN
+F 4 "SAM15910-ND" H 2200 1400 50  0001 C CNN "Digikey ID"
+F 5 "TSM-110-01-T-DH" H 2200 1400 50  0001 C CNN "MPN"
+F 6 "Samtec" H 2200 1400 50  0001 C CNN "Manufacturer"
+F 7 "https://www.digikey.com/en/products/detail/samtec-inc/TSM-110-01-T-DH/2685730" H 2200 1400 50  0001 C CNN "Ordering URL"
+F 8 "SMD" H 2200 1400 50  0001 C CNN "Type"
 	1    2200 1400
 	1    0    0    -1
@@
 F 1 "Conn_02x10_Odd_Even" H 2250 3450 50  0000 C CNN
 F 2 "Octopi:Samtec_TSM-110-01-X-DH_2x10_P2.54mm_Horizontal" H 2200 2900 50  0001 C CNN
-F 3 "~" H 2200 2900 50  0001 C CNN
+F 3 "http://suddendocs.samtec.com/catalog_english/tsm.pdf" H 2200 2900 50  0001 C CNN
+F 4 "SAM15910-ND" H 2200 2900 50  0001 C CNN "Digikey ID"
+F 5 "TSM-110-01-T-DH" H 2200 2900 50  0001 C CNN "MPN"
+F 6 "Samtec" H 2200 2900 50  0001 C CNN "Manufacturer"
+F 7 "https://www.digikey.com/en/products/detail/samtec-inc/TSM-110-01-T-DH/2685730" H 2200 2900 50  0001 C CNN "Ordering URL"
+F 8 "SMD" H 2200 2900 50  0001 C CNN "Type"
 	1    2200 2900
 	1    0    0    -1
@@
 F 1 "Conn_02x10_Odd_Even" H 2250 4950 50  0000 C CNN
 F 2 "Octopi:Samtec_TSM-110-01-X-DH_2x10_P2.54mm_Horizontal" H 2200 4400 50  0001 C CNN
-F 3 "~" H 2200 4400 50  0001 C CNN
+F 3 "http://suddendocs.samtec.com/catalog_english/tsm.pdf" H 2200 4400 50  0001 C CNN
+F 4 "SAM15910-ND" H 2200 4400 50  0001 C CNN "Digikey ID"
+F 5 "TSM-110-01-T-DH" H 2200 4400 50  0001 C CNN "MPN"
+F 6 "Samtec" H 2200 4400 50  0001 C CNN "Manufacturer"
+F 7 "https://www.digikey.com/en/products/detail/samtec-inc/TSM-110-01-T-DH/2685730" H 2200 4400 50  0001 C CNN "Ordering URL"
+F 8 "SMD" H 2200 4400 50  0001 C CNN "Type"
 	1    2200 4400
 	1    0    0    -1
