File: ODSv1.0.0-BP-Jmp/Connectors.sch (KiCad schematic (older format))
At the start: 2 parts, among them J2 Conn_02x60_Odd_Even, J3 Conn_02x60_Odd_Even

Commit message: Fix implementation of SPI CS multiplexing system (#22)
* Disconnect PP-T41's MAX7317's DOUT, since it's not needed anyways (#16)

* Disconnect BT & BP-Jmp backbone MAX7317 DOUT (#16); make DOUT output pin

* Replace DAC with a second MAX7317 expander with pullup resistors

* Insert 3-state buffers between MAX7317 DOUTs and CIPO in BP-Jmp (#16)

* Update symbol fields for I/O expansion components in BP-Jmp

* Consolidate free space by moving the AD7689 chip

* Add pull-ups on demuxed DCS (#17), move pull-ups to bottom of BP-Jmp

* Insert 3-state buffers between all MAX7317 DOUTs and CIPO (#16)

* Add bypass caps to the 3-state buffers for BP-Jmp's I/O expanders

* Fix title block for SPI DCS Selector sheet in BP-Jmp

* Use 2k pullups instead of 20k pullups on BP-Jmp

* Add 2k pullups on demuxed DSCS pins in PP-T41

* Define a NoPufferfish BOM variant of PP-T41

* Adjust the 12V copper fills on PP-T41

* Add 2k pullups within the DSCS selector in PP-T41 (#17)

* Add more information to READMEs

* Add 2k pullups within DCS selectors (#17), bump BP-Jmp to 0.2.0

* Fix errors in PR template for modified boards

* Move usage on I/O peripherals into a subsection in BP-Jmp's README.md

* Update KiCad preview & mechanical renders of all boards

* Improve & consolidate pull request templates

* Update raytrace renders of the entire stack

* Add missing definition for NoPufferfish variant for PP-T41

* Add link to CADLab project for this repo

* Remove the message annoyingly added by CADLab to top of README.md
Parts:
- renumbered J2 to J1, J3 to J2
Changed lines of the file:
@@
 $Descr USLetter 11000 8500
 encoding utf-8
-Sheet 4 9
+Sheet 3 9
 Title "Breakout Plane for Jumper Wires"
-Date "2021-03-09"
-Rev "v0.1.1"
+Date "2021-03-11"
+Rev "v0.2.0"
 Comp "Prakash Lab/Octopi Team"
 Comment1 "Designer: Ethan Li"
@@
 AR Path="/60EAE366" Ref="J?"  Part="1"
 AR Path="/60C51399/60EAE366" Ref="J?"  Part="1"
-AR Path="/60C51399/60E9531F/60EAE366" Ref="J2"  Part="1"
-F 0 "J2" H 2500 7067 50  0000 C CNN
+AR Path="/60C51399/60E9531F/60EAE366" Ref="J1"  Part="1"
+F 0 "J1" H 2500 7067 50  0000 C CNN
 F 1 "Conn_02x60_Odd_Even" H 2500 6976 50  0000 C CNN
 F 2 "Backbone_Connector_Hirose:Hirose_FX20_FX20-120P-0.5SV_2x60_P0.50mm_Vertical" H 2450 3950 50  0001 C CNN
@@
 AR Path="/61296724" Ref="J?"  Part="1"
 AR Path="/60C51399/61296724" Ref="J?"  Part="1"
-AR Path="/60C51399/60E9531F/61296724" Ref="J3"  Part="1"
-F 0 "J3" H 5500 7067 50  0000 C CNN
+AR Path="/60C51399/60E9531F/61296724" Ref="J2"  Part="1"
+F 0 "J2" H 5500 7067 50  0000 C CNN
 F 1 "Conn_02x60_Odd_Even" H 5500 6976 50  0000 C CNN
 F 2 "Backbone_Connector_Hirose:Hirose_FX20_FX20-120S-0.5SV_2x60_P0.50mm_Vertical" H 5450 3950 50  0001 C CNN
